File: pcb/pmw3610-xxs-compliant-narrow/pmw3610-xxs-compliant-narrow.kicad_sch (KiCad schematic)
At the start: 13 parts, among them J2 vik-module-connector, U1 MCP1700T-1802E/TT, U2 PMW3610

Commit message: Change VIK connector on trackball sensor module.
Parts:
- added H1, H2, H3: MountingHole_Pad, MountingHole:MountingHole_2.2mm_M2_Pad, symbol Mechanical:MountingHole_Pad
- C1, C2, C3, C4, C5, C6, C7, C8, C9: footprint roBa:C_0603_1608Metric -> Capacitor_SMD:C_0603_1608Metric_Pad1.08x0.95mm_HandSolder
- J2: footprint vik:vik-module-connector-vertical -> vik:vik-module-connector-horizontal-mini
- R1: footprint roBa:R_0603_1608Metric -> Resistor_SMD:R_0603_1608Metric_Pad0.98x0.95mm_HandSolder
- U1: footprint roBa:SOT-23 -> Package_TO_SOT_SMD:SOT-23
Connections:
- net GND: now also H1.1, H2.1, H3.1
Other:
- moved on the sheet: C1, C2, C3, C4, C5, C6, C7, C8, C9, J2, R1, U1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
