File: pcb/pmw3610-xxs-compliant-narrow/pmw3610-xxs-compliant-narrow.kicad_sch (KiCad schematic)
At the start: 16 parts, among them J2 vik-module-connector, U1 MCP1700T-1802E/TT, U2 PMW3610

Commit message: Add LCSC part numbers to pmw3610-narrow.
Parts:
- C1: LCSC C14663 -> C15849
- C3, C5, C8: LCSC C19666 -> C14663
- C4, C7: LCSC C19666 -> C57112
- C6: LCSC C19666 -> C19702
- C9: LCSC C19666 -> C51412
- J2: LCSC (none) -> C5213732
- R1: LCSC (none) -> C2930148
- U1: value MCP1700T-1802E/TT -> MG6208T3-18; LCSC (none) -> C22395363
Changed lines of the file:
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@@
 			)
 		)
-		(property "Value" "MCP1700T-1802E/TT"
+		(property "Value" "MG6208T3-18"
 			(at 45.72 27.178 0)
 			(show_name no)
@@
 			)
 		)
+		(property "LCSC" "C22395363"
+			(at 45.72 30.988 0)
+			(hide yes)
+			(show_name no)
+			(do_not_autoplace no)
+			(effects
+				(font
+					(size 1.27 1.27)
+				)
+			)
+		)
 		(pin "2"
 		)
@@
 			)
 		)
-		(property "LCSC" "C19666"
+		(property "LCSC" "C14663"
 			(at 99.06 44.958 0)
 			(hide yes)
@@
 			)
 		)
-		(property "LCSC" "C19666"
+		(property "LCSC" "C14663"
 			(at 171.45 34.798 0)
 			(hide yes)
@@
 			)
 		)
-		(property "LCSC" "C19666"
+		(property "LCSC" "C57112"
 			(at 154.94 24.638 0)
 			(hide yes)
@@
 			)
 		)
-		(property "LCSC" "C19666"
+		(property "LCSC" "C14663"
 			(at 154.94 38.608 0)
 			(hide yes)
@@
 			)
 		)
-		(property "LCSC" "C14663"
+		(property "LCSC" "C15849"
 			(at 34.29 33.528 0)
 			(hide yes)
@@
 		(property "Description" ""
 			(at 104.648 57.15 0)
+			(hide yes)
+			(show_name no)
+			(do_not_autoplace no)
+			(effects
+				(font
+					(size 1.27 1.27)
+				)
+			)
+		)
+		(property "LCSC" "C2930148"
+			(at 104.648 57.15 90)
 			(hide yes)
 			(show_name no)
@@
 			)
 		)
-		(property "LCSC" "C19666"
+		(property "LCSC" "C57112"
 			(at 170.18 51.308 0)
 			(hide yes)
@@
 			)
 		)
-		(property "LCSC" "C19666"
+		(property "LCSC" "C51412"
 			(at 179.07 34.798 0)
 			(hide yes)
@@
 			)
 		)
-		(property "LCSC" "C19666"
+		(property "LCSC" "C19702"
 			(at 162.56 51.308 0)
 			(hide yes)
@@
 			(at 48.26 81.788 0)
 			(hide yes)
+			(show_name no)
+			(do_not_autoplace no)
+			(effects
+				(font
+					(size 1.27 1.27)
+				)
+			)
+		)
+		(property "LCSC" "C5213732"
+			(at 48.26 81.788 0)
+			(hide yes)
