File: pcb/pmw3610-xxs-compliant-narrow/pmw3610-xxs-compliant-narrow.kicad_pcb (KiCad board)
At the start: 2 copper layers, 15 x 42 mm, 21 parts, among them J2 vik-module-connector, U1 MCP1700T-1802E/TT, U2 PMW3610

Commit message: Add LCSC part numbers to pmw3610-narrow.
Parts:
- removed the REF** at (33.0, 30.0)
- C1, C2, C3, C5, C8, C9, R1: moved to F.Cu
- U1: value MCP1700T-1802E/TT -> MG6208T3-18
- moved C2 26.3 mm to (31.5, 28.0), turned to 90 degrees
- moved C8 26.3 mm to (34.5, 28.0), turned to 90 degrees
- moved C9 26.3 mm to (33.0, 28.0), turned to 90 degrees
- moved C1 26.2 mm to (24.5, 28.0)
- moved C3 26.2 mm to (23.0, 28.0)
- moved R1 26.2 mm to (21.5, 28.0)
- moved U1 20.5 mm to (33.5, 34.0), turned to 90 degrees
- moved C4 5.42 mm to (29.0, 55.0)
- moved C5 2.64 mm to (31.0, 55.0)
- moved C7 0.93 mm to (27.0, 55.0)
- moved C6 0.87 mm to (25.0, 55.0)
- moved J2 0.19 mm to (28.0, 32.4)
Routing:
- net VCC: track 61.6 -> 34.6 mm, vias 2 -> 3
- net Net-(U2-NRESET): track 7.73 -> 20.6 mm, vias 0 -> 1
- net GND: track 71.4 -> 80.4 mm, vias 6 -> 2
- net SDIO: track 16.2 -> 12.8 mm
- net Net-(U2-CP): track 8.55 -> 11.3 mm, vias 1 -> 0
- net +1V9: track 19.3 -> 16.9 mm, vias 1 -> 0
- net Net-(U2-CN): track 12.3 -> 14.4 mm, vias 1 -> 0
- net NCS: track 19.2 -> 18.3 mm
- net SCLK: track 15.9 -> 16.4 mm, vias 0 -> 1
- net MOTION: track 26.1 -> 25.7 mm, vias 2 -> 0

Commit message: Add more ground vias to PMW3610-narrow.
Routing:
- net GND: vias 2 -> 6
Changed lines of the file:
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@@
 		(capping no)
 		(filling no)
-		(zone_defaults)
 		(pcbplotparams
 			(layerselection 0x00000000_00000000_55555555_5755f5ff)
@@
 				(font
 					(size 1.27 1.27)
+					(thickness 0.15)
 				)
 			)
@@
 				(font
 					(size 1.27 1.27)
+					(thickness 0.15)
 				)
 			)
@@
 				(font
 					(size 1.27 1.27)
+					(thickness 0.15)
 				)
 			)
@@
 				(font
 					(size 1.27 1.27)
+					(thickness 0.15)
 				)
 			)
@@
 	)
 	(via
+		(at 34 55)
+		(size 0.6)
+		(drill 0.3)
+		(layers "F.Cu" "B.Cu")
+		(net "GND")
+	)
+	(via
+		(at 22 55)
+		(size 0.6)
+		(drill 0.3)
+		(layers "F.Cu" "B.Cu")
+		(free yes)
+		(net "GND")
+	)
+	(via
+		(at 34.5 27.1375)
+		(size 0.6)
+		(drill 0.3)
+		(layers "F.Cu" "B.Cu")
+		(net "GND")
+	)
+	(via
 		(at 29 55.8625)
 		(size 0.6)
@@
 		(net "GND")
 	)
+	(via
+		(at 23 28.8625)
+		(size 0.6)
+		(drill 0.3)
+		(layers "F.Cu" "B.Cu")
+		(net "GND")
+	)
 	(segment
-		(start 29 55.8625)
-		(end 33.6375 55.8625)
+		(start 35.35 33.993261)
+		(end 33.769239 32.4125)
 		(width 0.3)
 		(layer "B.Cu")
@@
 	)
 	(segment
-		(start 33.769239 32.4125)
-		(end 26.4375 32.4125)
+		(start 34.25 55.25)
+		(end 33.6375 55.8625)
 		(width 0.3)
 		(layer "B.Cu")
@@
 	(segment
 		(start 33.6375 55.8625)
+		(end 29 55.8625)
+		(width 0.3)
+		(layer "B.Cu")
+		(net "GND")
+	)
+	(segment
+		(start 34.25 55.25)
 		(end 35.35 54.15)
 		(width 0.3)
@@
 	)
 	(segment
-		(start 26.4375 32.4125)
-		(end 26 32.85)
+		(start 35.35 54.15)
+		(end 35.35 33.993261)
 		(width 0.3)
 		(layer "B.Cu")
@@
 	)
 	(segment
-		(start 35.35 33.993261)
-		(end 33.769239 32.4125)
+		(start 26.4375 32.4125)
+		(end 26 32.85)
 		(width 0.3)
 		(layer "B.Cu")
@@
 	)
 	(segment
-		(start 35.35 54.15)
-		(end 35.35 33.993261)
+		(start 33.769239 32.4125)
+		(end 26.4375 32.4125)
 		(width 0.3)
 		(layer "B.Cu")
@@
 	)
 	(segment
+		(start 33 28.8625)
+		(end 34.5 28.8625)
+		(width 0.3)
+		(layer "F.Cu")
+		(net "+1V9")
+	)
+	(segment
+		(start 34.45 34.9375)
+		(end 34.45 41.17)
+		(width 0.3)
+		(layer "F.Cu")
+		(net "+1V9")
+	)
+	(segment
+		(start 34.45 41.17)
+		(end 33.35 42.27)
+		(width 0.3)
+		(layer "F.Cu")
+		(net "+1V9")
+	)
+	(segment
+		(start 31.5 28.8625)
+		(end 33 28.8625)
+		(width 0.3)
+		(layer "F.Cu")
+		(net "+1V9")
+	)
+	(segment
+		(start 34.5 29)
+		(end 34.45 29.05)
+		(width 0.3)
+		(layer "F.Cu")
+		(net "+1V9")
+	)
+	(segment
+		(start 34.5 28.8625)
+		(end 34.5 29)
+		(width 0.3)
+		(layer "F.Cu")
+		(net "+1V9")
+	)
+	(segment
+		(start 34.45 29.05)
+		(end 34.45 34.9375)
+		(width 0.3)
+		(layer "F.Cu")
+		(net "+1V9")
+	)
+	(segment
 		(start 28.3375 52.8)
 		(end 27 54.1375)
@@
 		(net "Net-(U2-VCP)")
 	)
+	(segment
+		(start 33.35 44.05)
+		(end 35.175 45.875)
+		(width 0.2)
+		(layer "F.Cu")
+		(net "Net-(U2-CN)")
+	)
+	(segment
+		(start 31.238441 55.8625)
+		(end 31 55.8625)
+		(width 0.2)
+		(layer "F.Cu")
+		(net "Net-(U2-CN)")
+	)
+	(segment
+		(start 35.175 45.875)
+		(end 35.175 51.925941)
+		(width 0.2)
+		(layer "F.Cu")
+		(net "Net-(U2-CN)")
+	)
+	(segment
+		(start 35.175 51.925941)
+		(end 31.238441 55.8625)
+		(width 0.2)
+		(layer "F.Cu")
+		(net "Net-(U2-CN)")
+	)
+	(segment
+		(start 34.775 51.760255)
+		(end 32.397755 54.1375)
+		(width 0.2)
+		(layer "F.Cu")
+		(net "Net-(U2-CP)")
+	)
+	(segment
+		(start 32.397755 54.1375)
+		(end 31 54.1375)
+		(width 0.2)
+		(layer "F.Cu")
+		(net "Net-(U2-CP)")
+	)
+	(segment
+		(start 34.775 47.255)
+		(end 34.775 51.760255)
+		(width 0.2)
+		(layer "F.Cu")
+		(net "Net-(U2-CP)")
+	)
+	(segment
+		(start 33.35 45.83)
+		(end 34.775 47.255)
+		(width 0.2)
+		(layer "F.Cu")
+		(net "Net-(U2-CP)")
+	)
 	(via
 		(at 29 54.1375)
@@
 	)
 	(segment
-		(start 34.775 51.760255)
-		(end 32.397755 54.1375)
-		(width 0.2)
-		(layer "F.Cu")
-		(net "Net-(U2-CP)")
-	)
-	(segment
-		(start 32.397755 54.1375)
-		(end 31 54.1375)
-		(width 0.2)
-		(layer "F.Cu")
-		(net "Net-(U2-CP)")
-	)
-	(segment
-		(start 34.775 47.255)
-		(end 34.775 51.760255)
-		(width 0.2)
-		(layer "F.Cu")
-		(net "Net-(U2-CP)")
-	)
-	(segment
-		(start 33.35 45.83)
-		(end 34.775 47.255)
-		(width 0.2)
-		(layer "F.Cu")
-		(net "Net-(U2-CP)")
-	)
-	(segment
-		(start 33.35 44.05)
-		(end 35.175 45.875)
-		(width 0.2)
-		(layer "F.Cu")
-		(net "Net-(U2-CN)")
-	)
-	(segment
-		(start 31.238441 55.8625)
-		(end 31 55.8625)
-		(width 0.2)
-		(layer "F.Cu")
-		(net "Net-(U2-CN)")
-	)
-	(segment
-		(start 35.175 45.875)
-		(end 35.175 51.925941)
-		(width 0.2)
-		(layer "F.Cu")
-		(net "Net-(U2-CN)")
-	)
-	(segment
-		(start 35.175 51.925941)
-		(end 31.238441 55.8625)
-		(width 0.2)
-		(layer "F.Cu")
-		(net "Net-(U2-CN)")
-	)
-	(segment
-		(start 33 28.8625)
-		(end 34.5 28.8625)
-		(width 0.3)
-		(layer "F.Cu")
-		(net "+1V9")
-	)
-	(segment
-		(start 34.45 34.9375)
-		(end 34.45 41.17)
-		(width 0.3)
-		(layer "F.Cu")
-		(net "+1V9")
-	)
-	(segment
-		(start 34.45 41.17)
-		(end 33.35 42.27)
-		(width 0.3)
-		(layer "F.Cu")
-		(net "+1V9")
-	)
-	(segment
-		(start 31.5 28.8625)
-		(end 33 28.8625)
-		(width 0.3)
-		(layer "F.Cu")
-		(net "+1V9")
-	)
-	(segment
-		(start 34.5 29)
-		(end 34.45 29.05)
-		(width 0.3)
-		(layer "F.Cu")
-		(net "+1V9")
-	)
-	(segment
-		(start 34.5 28.8625)
-		(end 34.5 29)
-		(width 0.3)
-		(layer "F.Cu")
-		(net "+1V9")
-	)
-	(segment
-		(start 34.45 29.05)
-		(end 34.45 34.9375)
-		(width 0.3)
-		(layer "F.Cu")
-		(net "+1V9")
-	)
-	(segment
